Commit message: diff drive integration

File: robot_description/urdf/robot.xacro (robot description, xacro)
@@ -31,4 +31,5 @@
     <xacro:property name="caster" value = "${config['caster']}"/>
   </xacro:if>
+  <xacro:include filename="$(find robot_description)/urdf/robot.gazebo" />
   <xacro:include filename="$(find robot_description)/urdf/body.xacro" />
   <xacro:include filename="$(find robot_description)/urdf/wheel.xacro" />

File: robot_description/urdf/wheel.xacro (robot description, xacro)
@@ -2,5 +2,5 @@
 <robot name="wheel" xmlns:xacro="http://www.ros.org/wiki/xacro">
   <xacro:macro name="wheel" params="lr flip">
-    <link name="${lr}_wheel">
+    <link name="${lr}_wheel_link">
       <visual>
         <origin xyz="0 0 0" rpy="${M_PI_2} 0 0" />
@@ -22,5 +22,5 @@
       </inertial>
     </link>
-    <gazebo reference="${lr}_wheel">
+    <gazebo reference="${lr}_wheel_link">
       <mu1 value="0.01"/>
       <mu2 value="1.0"/>
@@ -32,7 +32,7 @@
       <turnGravityOff>false</turnGravityOff>
     </gazebo>
-    <joint name="$base_to_${lr}_wheel" type="continuous">
+    <joint name="${lr}_wheel_joint" type="continuous">
       <parent link="base_link"/>
-      <child link="${lr}_wheel"/>
+      <child link="${lr}_wheel_link"/>
       <origin xyz="0 ${flip * (body['width']/2 + wheel['length']/2)} 0" rpy="0 0 0"/>
       <axis xyz="0 1 0" />
@@ -40,4 +40,26 @@
       <joint_properties damping="0.0" friction="0.0"/>
     </joint>
+    <!-- Orientation transmission for the steering -->
+    <!-- <transmission name="${lr}_wheel_joint_pos_trans">
+    <type>transmission_interface/SimpleTransmission</type>
+        <joint name="${lr}_wheel_joint">
+            <hardwareInterface>hardware_interface/EffortJointInterface</hardwareInterface>
+        </joint>
+        <actuator name="${lr}_wheel_joint_motor">
+            <hardwareInterface>hardware_interface/EffortJointInterface</hardwareInterface>
+            <mechanicalReduction>1</mechanicalReduction>
+        </actuator>
+    </transmission> -->
+    <!-- Wheel velocity transmission -->
+    <transmission name="${lr}_wheel_joint_vel_trans">
+    <type>transmission_interface/SimpleTransmission</type>
+        <joint name="${lr}_wheel_joint">
+            <hardwareInterface>hardware_interface/VelocityJointInterface</hardwareInterface>
+        </joint>
+        <actuator name="${lr}_wheel_joint_motor">
+            <hardwareInterface>hardware_interface/VelocityJointInterface</hardwareInterface>
+            <mechanicalReduction>1</mechanicalReduction>
+        </actuator>
+    </transmission>
   </xacro:macro>
 </robot>
