Commit message: Adding inertias

File: robot_description/urdf/body.xacro (robot description, xacro)
@@ -12,4 +12,8 @@
             </geometry>
         </collision>
+        <inertial>
+        <mass value="5" />
+        <inertia ixx="0.004" ixy="0.001" ixz="0" iyy="0.006" iyz="0" izz="0.007" />
+        </inertial>
     </link>
     <joint name="body_joint" type="fixed">

File: robot_description/urdf/caster.xacro (robot description, xacro)
@@ -25,4 +25,8 @@
       </surface>
     </collision>
+    <inertial>
+    <mass value="5" />
+    <inertia ixx="0.004" ixy="0.001" ixz="0" iyy="0.006" iyz="0" izz="0.007" />
+    </inertial>
   </link>
   <joint name="caster_joint" type="fixed">

File: robot_description/urdf/wheel.xacro (robot description, xacro)
@@ -7,7 +7,16 @@
                 <geometry>
                 <!-- TODO: parametrizar valores -->
-                <cylinder radius="0.1" length="0.05"/>
+                <cylinder radius="wheel['radius']" length="wheel['length']"/>
                 </geometry>
             </visual>
+            <collision>
+                <geometry>
+                <cylinder radius="wheel['radius']" length="wheel['length']"/>
+                </geometry>
+            </collision>
+            <inertial>
+            <mass value="5" />
+            <inertia ixx="0.004" ixy="0.001" ixz="0" iyy="0.006" iyz="0" izz="0.007" />
+            </inertial>
         </link>
         <joint name="$base_to_${lr}_wheel" type="continuous">

Commit message: Inertias properly placed. Model can be pushed in Gazebo

File: robot_description/urdf/body.xacro (robot description, xacro)
@@ -1,47 +1,28 @@
 <?xml version="1.0"?>
 <robot name="body" xmlns:xacro="http://www.ros.org/wiki/xacro">
-    <link name="body_link">
-        <visual name="visual">
-            <geometry>
-            <box size="${body['length']} ${body['width']} ${body['height']}"/>
-            </geometry>
-        </visual>
-        <collision name="collision">
-            <geometry>
-            <box size="${body['length']} ${body['width']} ${body['height']}"/>
-            </geometry>
-        </collision>
-        <inertial>
-        <mass value="5" />
-        <inertia ixx="0.004" ixy="0.001" ixz="0" iyy="0.006" iyz="0" izz="0.007" />
-        </inertial>
-    </link>
-    <joint name="body_joint" type="fixed">
-        <parent link="base_link" />
-        <child link="body_link" />
-        <origin xyz="${body['length']/2} 0 0" />
-    </joint>
-    <!-- Wheel links -->
-    <link name="back_left_wheel_link">
-    </link>
-    <joint name="back_left_wheel_joint" type="fixed">
-        <parent link="base_link" />
-        <child link="back_left_wheel_link" />
-        <origin xyz="0 ${body['width']/2 + wheel['length']/2} 0" rpy="-${M_PI_2} 0 0"/>
-    </joint>
-    <link name="back_right_wheel_link">
-    </link>
-    <joint name="back_right_wheel_joint" type="fixed">
-        <parent link="base_link" />
-        <child link="back_right_wheel_link" />
-        <origin xyz="0 -${body['width']/2 + wheel['length']/2} 0" rpy="${M_PI_2} 0 0"/>
-    </joint>
-    <!-- Caster link -->
-    <link name="base_to_caster_link">
-    </link>
-    <joint name="base_to_caster_joint" type="fixed">
-        <parent link="base_link" />
-        <child link="base_to_caster_link" />
-        <origin xyz="0.35 0 -${caster['radius']}" rpy="0 0 0"/>
-    </joint>
+  <link name="body_link">
+    <visual name="visual">
+      <geometry>
+      <box size="${body['length']} ${body['width']} ${body['height']}"/>
+      </geometry>
+    </visual>
+    <collision name="collision">
+      <geometry>
+      <box size="${body['length']} ${body['width']} ${body['height']}"/>
+      </geometry>
+    </collision>
+    <inertial>
+      <mass value="5" />
+      <box_inertia m="5" x="${body['length']}" y="${body['width']}" z="${body['height']}" />
+    </inertial>
+  </link>
+  <gazebo reference="body_link">
+    <material>Gazebo/Yellow</material>
+    <turnGravityOff>false</turnGravityOff>
+  </gazebo>
+  <joint name="body_joint" type="fixed">
+    <parent link="base_link" />
+    <child link="body_link" />
+    <origin xyz="${body['length']/2} 0 0" />
+  </joint>
 </robot>

File: robot_description/urdf/caster.xacro (robot description, xacro)
@@ -14,24 +14,26 @@
       <sphere radius="${caster['radius']}"/>
       </geometry>
-      <surface>
-        <friction>
-          <ode>
-            <mu>0</mu>
-            <mu2>0</mu2>
-            <slip1>1.0</slip1>
-            <slip2>1.0</slip2>
-          </ode>
-        </friction>
-      </surface>
     </collision>
     <inertial>
-    <mass value="5" />
-    <inertia ixx="0.004" ixy="0.001" ixz="0" iyy="0.006" iyz="0" izz="0.007" />
+      <mass value="1" />
+      <sphere_inertia m="1" r="${wheel['radius']}" />
     </inertial>
   </link>
-  <joint name="caster_joint" type="fixed">
-    <parent link="base_to_caster_link"/>
+  <gazebo reference="caster_link">
+    <mu1 value="0.0"/>
+    <mu2 value="1.0"/>
+    <kp  value="10000000.0"/>
+    <kd  value="1.0" />
+    <fdir1 value="0 1 0"/>
+    <minDepth value="0.001"/>
+    <material>Gazebo/Black</material>
+    <turnGravityOff>false</turnGravityOff>
+  </gazebo>
+  <joint name="caster_joint" type="continuous">
+    <parent link="base_link"/>
     <child link="$caster_link"/>
-    <origin xyz="0 0 0" />
+    <origin xyz="0.35 0 -${caster['radius']}" rpy="0 0 0"/>
+    <axis xyz="0 1 0" />
+    <joint_properties damping="0.0" friction="0.0"/>
   </joint>
 </robot>

File: robot_description/urdf/robot.xacro (robot description, xacro)
@@ -3,4 +3,20 @@
   <property name="M_PI" value="3.1415926535897931" />
   <property name="M_PI_2" value="1.570796327" />
+  <!-- Macro for calculating inertia of cylinder -->
+  <macro name="cylinder_inertia" params="m r h">
+    <inertia  ixx="${m*(3*r*r+h*h)/12}" ixy = "0" ixz = "0"
+              iyy="${m*(3*r*r+h*h)/12}" iyz = "0"
+              izz="${m*r*r/2}" />
+  </macro>
+  <macro name="box_inertia" params="m x y z">
+    <inertia  ixx="${m*(y*y+z*z)/12}" ixy = "0" ixz = "0"
+              iyy="${m*(x*x+z*z)/12}" iyz = "0"
+              izz="${m*(x*x+y*y)/12}" />
+  </macro>
+  <macro name="sphere_inertia" params="m r">
+    <inertia  ixx="${2*m*r*r/5}" ixy = "0" ixz = "0"
+              iyy="${2*m*r*r/5}" iyz = "0"
+              izz="${2*m*r*r/5}" />
+  </macro>
   <xacro:property name="config_file"
                  value="$(find robot_description)/urdf/config/config.yaml"/>
@@ -20,7 +36,11 @@
   <link name="base_link">
   </link>
+  <gazebo reference="base_link">
+    <material>Gazebo/Yellow</material>
+    <turnGravityOff>false</turnGravityOff>
+  </gazebo>
   <body/>
   <caster/>
-  <wheel lr="left"/>
-  <wheel lr="right"/>
+  <wheel lr="left" flip="1"/>
+  <wheel lr="right" flip="-1"/>
 </robot>

File: robot_description/urdf/wheel.xacro (robot description, xacro)
@@ -1,28 +1,43 @@
 <?xml version="1.0"?>
 <robot name="wheel" xmlns:xacro="http://www.ros.org/wiki/xacro">
-    <xacro:macro name="wheel" params="lr">
-        <link name="${lr}_wheel">
-            <visual>
-                <origin xyz="0 0 0" rpy="0 0 0" />
-                <geometry>
-                <!-- TODO: parametrizar valores -->
-                <cylinder radius="wheel['radius']" length="wheel['length']"/>
-                </geometry>
-            </visual>
-            <collision>
-                <geometry>
-                <cylinder radius="wheel['radius']" length="wheel['length']"/>
-                </geometry>
-            </collision>
-            <inertial>
-            <mass value="5" />
-            <inertia ixx="0.004" ixy="0.001" ixz="0" iyy="0.006" iyz="0" izz="0.007" />
-            </inertial>
-        </link>
-        <joint name="$base_to_${lr}_wheel" type="continuous">
-            <parent link="back_${lr}_wheel_link"/>
-            <child link="${lr}_wheel"/>
-            <origin xyz="0 0 0" />
-        </joint>
-    </xacro:macro>
+  <xacro:macro name="wheel" params="lr flip">
+    <link name="${lr}_wheel">
+      <visual>
+        <origin xyz="0 0 0" rpy="${M_PI_2} 0 0" />
+        <geometry>
+        <!-- TODO: parametrizar valores -->
+        <cylinder radius="${wheel['radius']}" length="${wheel['length']}"/>
+        </geometry>
+      </visual>
+      <collision>
+        <origin xyz="0 0 0" rpy="${M_PI_2} 0 0" />
+        <geometry>
+        <cylinder radius="${wheel['radius']}" length="${wheel['length']}"/>
+        </geometry>
+      </collision>
+      <inertial>
+        <origin xyz="0 0 0" rpy="${M_PI_2} 0 0" />
+        <mass value="1" />
+        <cylinder_inertia m="1" r="${wheel['radius']}" h="${wheel['length']}" />
+      </inertial>
+    </link>
+    <gazebo reference="${lr}_wheel">
+      <mu1 value="0.01"/>
+      <mu2 value="1.0"/>
+      <kp  value="10000000.0"/>
+      <kd  value="1.0" />
+      <fdir1 value="1 0 0"/>
+      <minDepth value="0.001"/>
+      <material>Gazebo/Grey</material>
+      <turnGravityOff>false</turnGravityOff>
+    </gazebo>
+    <joint name="$base_to_${lr}_wheel" type="continuous">
+      <parent link="base_link"/>
+      <child link="${lr}_wheel"/>
+      <origin xyz="0 ${flip * (body['width']/2 + wheel['length']/2)} 0" rpy="0 0 0"/>
+      <axis xyz="0 1 0" />
+      <limit effort="100000000" velocity="2"/>
+      <joint_properties damping="0.0" friction="0.0"/>
+    </joint>
+  </xacro:macro>
 </robot>

Commit message: Added base_footprint

File: robot_description/urdf/body.xacro (robot description, xacro)
@@ -1,4 +1,33 @@
 <?xml version="1.0"?>
 <robot name="body" xmlns:xacro="http://www.ros.org/wiki/xacro">
+  <link name="base_link">
+    <inertial>
+    <mass value="0.0001" />
+    <inertia ixx="0.0001" ixy="0.0" ixz="0.0"
+      iyy="0.0001" iyz="0.0"
+      izz="0.0001" />
+    </inertial>
+    <origin xyz="0 0 0" rpy="0 0 0" />
+  </link>
+  <gazebo reference="base_link">
+    <material>Gazebo/Yellow</material>
+    <turnGravityOff>false</turnGravityOff>
+  </gazebo>
+  <link name="base_footprint">
+    <inertial>
+      <mass value="0.0001" />
+      <inertia ixx="0.0001" ixy="0.0" ixz="0.0"
+          iyy="0.0001" iyz="0.0"
+          izz="0.0001" />
+      </inertial>
+  </link>
+  <joint name="base_footprint_joint" type="fixed">
+      <origin xyz="0 0 0.1" rpy="0 0 0" />
+      <parent link="base_footprint"/>
+      <child link="base_link" />
+  </joint>
+  <gazebo reference="base_footprint">
+      <turnGravityOff>false</turnGravityOff>
+  </gazebo>
   <link name="body_link">
     <visual name="visual">
@@ -13,6 +42,7 @@
     </collision>
     <inertial>
-      <mass value="5" />
-      <box_inertia m="5" x="${body['length']}" y="${body['width']}" z="${body['height']}" />
+      <mass value="20" />
+      <origin xyz="-0.05 0 0" rpy="0 0 0" />
+      <box_inertia m="20" x="${body['length']}" y="${body['width']}" z="${body['height']}" />
     </inertial>
   </link>

File: robot_description/urdf/robot.xacro (robot description, xacro)
@@ -35,10 +35,4 @@
   <xacro:include filename="$(find robot_description)/urdf/wheel.xacro" />
   <xacro:include filename="$(find robot_description)/urdf/caster.xacro" />
-  <link name="base_link">
-  </link>
-  <gazebo reference="base_link">
-    <material>Gazebo/Yellow</material>
-    <turnGravityOff>false</turnGravityOff>
-  </gazebo>
   <body/>
   <caster/>
