Commit message: Tuned wheels and caster values

File: robot_description/urdf/caster.xacro (robot description, xacro)
@@ -5,5 +5,4 @@
       <origin xyz="0 0 0" rpy="0 0 0" />
       <geometry>
-      <!-- TODO: parametrizar valores -->
       <sphere radius="${caster['radius']}"/>
       </geometry>
@@ -16,24 +15,25 @@
     </collision>
     <inertial>
-      <mass value="1" />
-      <sphere_inertia m="1" r="${wheel['radius']}" />
+      <mass value="${caster['mass']}"/>
+      <sphere_inertia m="${caster['mass']}" r="${caster['radius']}" />
     </inertial>
   </link>
   <gazebo reference="caster_link">
     <mu1 value="0.0"/>
-    <mu2 value="1.0"/>
-    <kp  value="10000000.0"/>
+    <mu2 value="0.0"/>
+    <kp  value="1000000.0"/>
     <kd  value="1.0" />
-    <fdir1 value="0 1 0"/>
-    <minDepth value="0.001"/>
+    <fdir1 value="1 1 1"/>
+    <minDepth value="0.0"/>
     <material>Gazebo/Black</material>
     <turnGravityOff>false</turnGravityOff>
   </gazebo>
-  <joint name="caster_joint" type="continuous">
+  <joint name="caster_joint" type="fixed">
     <parent link="base_link"/>
     <child link="$caster_link"/>
     <origin xyz="0.35 0 -${caster['radius']}" rpy="0 0 0"/>
-    <axis xyz="0 1 0" />
-    <joint_properties damping="0.0" friction="0.0"/>
+    <axis xyz="1 1 1" />
+    <limit effort="100" velocity="2"/>
+    <joint_properties damping="1.0" friction="0.0"/>
   </joint>
 </robot>

File: robot_description/urdf/wheel.xacro (robot description, xacro)
@@ -6,5 +6,4 @@
         <origin xyz="0 0 0" rpy="${M_PI_2} 0 0" />
         <geometry>
-        <!-- TODO: parametrizar valores -->
         <cylinder radius="${wheel['radius']}" length="${wheel['length']}"/>
         </geometry>
@@ -18,14 +17,14 @@
       <inertial>
         <origin xyz="0 0 0" rpy="${M_PI_2} 0 0" />
-        <mass value="1" />
-        <cylinder_inertia m="1" r="${wheel['radius']}" h="${wheel['length']}" />
+        <mass value="${wheel['mass']}" />
+        <cylinder_inertia m="${wheel['mass']}" r="${wheel['radius']}" h="${wheel['length']}" />
       </inertial>
     </link>
     <gazebo reference="${lr}_wheel_link">
-      <mu1 value="0.01"/>
-      <mu2 value="1.0"/>
-      <kp  value="10000000.0"/>
+      <mu1 value="50000000.0"/>
+      <mu2 value="10.0"/>
+      <kp  value="1000000000.0"/>
       <kd  value="1.0" />
-      <fdir1 value="1 0 0"/>
+      <fdir1 value="0 0 1"/>
       <minDepth value="0.001"/>
       <material>Gazebo/Grey</material>
@@ -35,20 +34,8 @@
       <parent link="base_link"/>
       <child link="${lr}_wheel_link"/>
-      <origin xyz="0 ${flip * (body['width']/2 + wheel['length']/2)} 0" rpy="0 0 0"/>
+      <origin xyz="0.02 ${flip * (body['width']/2 + wheel['length']/2)} 0" rpy="0 0 0"/>
       <axis xyz="0 1 0" />
-      <limit effort="100000000" velocity="2"/>
-      <joint_properties damping="0.0" friction="0.0"/>
+      <limit effort="5000000000" velocity="10"/>
     </joint>
-    <!-- Orientation transmission for the steering -->
-    <!-- <transmission name="${lr}_wheel_joint_pos_trans">
-    <type>transmission_interface/SimpleTransmission</type>
-        <joint name="${lr}_wheel_joint">
-            <hardwareInterface>hardware_interface/EffortJointInterface</hardwareInterface>
-        </joint>
-        <actuator name="${lr}_wheel_joint_motor">
-            <hardwareInterface>hardware_interface/EffortJointInterface</hardwareInterface>
-            <mechanicalReduction>1</mechanicalReduction>
-        </actuator>
-    </transmission> -->
     <!-- Wheel velocity transmission -->
     <transmission name="${lr}_wheel_joint_vel_trans">
